File: ipd_task1.kicad_pcb (KiCad board)
At the start: 2 copper layers, 82.5 x 93 mm, 37 parts, among them J1 Barrel_Jack, J10 C_02x03, J2 Barrel_Jack, J3 Conn_01x08, J4 Conn_01x08, J5 ST_01x02, J6 ST_01x02, J7 ST_01x06, J8 Conn_01x06, J9 Conn_01x08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

Commit message: Add files via upload
Routing:
- net GND: track 278.6 -> 26.3 mm, vias 5 -> 1
- added copper zone on B.Cu, net GND
